File: LoliBot.sch (KiCad schematic (older format))
At the start: 42 parts, among them J1 LOLINBATT, J10 LEFT-MOTOR, J11 REFLECT_, J12 MECH, J13 MECH, J14 MECH, J15 MECH, J16 MECH, J17 MECH, J18 MECH, J19 MECH, J2 APA106, J20 CONN_01X08, J21 CONN_01X08, J22 BRIDGE_RIGHT, J23 BRIDGE_LEFT, J24 FUSE_BRIDGE, J25 MECH, J26 MECH, J27 MECH, J28 MECH, J29 MECH, J3 SERVO1, J30 MECH, J31 LCA_LOGO, J32 FREETRONICS_LOGO, J4 RIGHT, J5 LEFT, J6 MPU-9250, J7 APA106, J8 APA106, J9 RIGHT-MOTOR, SW1 ON|OFF, U1 LOLIN32-LITE, U3 L9110, U4 L9110

Commit message: Added more text
Parts:
- BT1: value Battery_Cell -> BATTERY
Changed lines of the file:
@@
 P 1500 1450
 F 0 "BT1" H 1600 1550 50  0000 L CNN
-F 1 "Battery_Cell" H 1600 1450 50  0000 L CNN
+F 1 "BATTERY" H 1600 1450 50  0000 L CNN
 F 2 "libs:BH-18650" V 1500 1510 50  0001 C CNN
 F 3 "" V 1500 1510 50  0001 C CNN
@@
 	2800 1150 2850 1150
 Wire Wire Line
-	2850 1450 2850 1150
+	2850 1150 2850 1450
 Text Label 1350 1150 0    60   ~ 0
 BATT_V
@@
 $EndComp
 Wire Wire Line
-	2200 1450 2850 1450
+	2850 1450 2200 1450
 Wire Wire Line
 	1700 1450 1900 1450

Commit message: i2c pullup resistors
Parts:
- added R1, R2: 4K7, Resistors_SMD:R_0603_HandSoldering, symbol R
Connections:
- net +3V3: now also R1.1, R2.1
- net IO18: now also R2.2
- net IO19: now also R1.2
Changed lines of the file:
@@
 $EndComp
 $Comp
-L GND #PWR01
+L GND #PWR1
 U 1 1 59DB6136
 P 1250 2150
-F 0 "#PWR01" H 1250 1900 50  0001 C CNN
+F 0 "#PWR1" H 1250 1900 50  0001 C CNN
 F 1 "GND" H 1250 2000 50  0000 C CNN
 F 2 "" H 1250 2150 50  0001 C CNN
@@
 $EndComp
 $Comp
-L GND #PWR02
+L GND #PWR9
 U 1 1 59DB834E
 P 7200 1800
-F 0 "#PWR02" H 7200 1550 50  0001 C CNN
+F 0 "#PWR9" H 7200 1550 50  0001 C CNN
 F 1 "GND" H 7200 1650 50  0000 C CNN
 F 2 "" H 7200 1800 50  0001 C CNN
@@
 $EndComp
 $Comp
-L GND #PWR03
+L GND #PWR4
 U 1 1 59DBA675
 P 4300 3550
-F 0 "#PWR03" H 4300 3300 50  0001 C CNN
+F 0 "#PWR4" H 4300 3300 50  0001 C CNN
 F 1 "GND" H 4300 3400 50  0000 C CNN
 F 2 "" H 4300 3550 50  0001 C CNN
@@
 $EndComp
 $Comp
-L GND #PWR04
+L GND #PWR15
 U 1 1 59DBB61B
 P 10450 4750
-F 0 "#PWR04" H 10450 4500 50  0001 C CNN
+F 0 "#PWR15" H 10450 4500 50  0001 C CNN
 F 1 "GND" H 10450 4600 50  0000 C CNN
 F 2 "" H 10450 4750 50  0001 C CNN
@@
 $EndComp
 $Comp
-L GND #PWR05
+L GND #PWR16
 U 1 1 59DBCDC3
 P 10500 6200
-F 0 "#PWR05" H 10500 5950 50  0001 C CNN
+F 0 "#PWR16" H 10500 5950 50  0001 C CNN
 F 1 "GND" H 10500 6050 50  0000 C CNN
 F 2 "" H 10500 6200 50  0001 C CNN
@@
 $EndComp
 $Comp
-L GND #PWR06
+L GND #PWR12
 U 1 1 59DBDB38
 P 8400 3100
-F 0 "#PWR06" H 8400 2850 50  0001 C CNN
+F 0 "#PWR12" H 8400 2850 50  0001 C CNN
 F 1 "GND" H 8400 2950 50  0000 C CNN
 F 2 "" H 8400 3100 50  0001 C CNN
@@
 IO13
 $Comp
-L +3.3V #PWR07
+L +3.3V #PWR3
 U 1 1 59DC0699
 P 3300 4450
-F 0 "#PWR07" H 3300 4300 50  0001 C CNN
+F 0 "#PWR3" H 3300 4300 50  0001 C CNN
 F 1 "+3.3V" H 3300 4590 50  0000 C CNN
 F 2 "" H 3300 4450 50  0001 C CNN
@@
 $EndComp
 $Comp
-L GND #PWR08
+L GND #PWR2
 U 1 1 59DC0B2B
 P 1300 6000
-F 0 "#PWR08" H 1300 5750 50  0001 C CNN
+F 0 "#PWR2" H 1300 5750 50  0001 C CNN
 F 1 "GND" H 1300 5850 50  0000 C CNN
 F 2 "" H 1300 6000 50  0001 C CNN
@@
 FSYNC
 $Comp
-L +3.3V #PWR09
+L +3.3V #PWR13
 U 1 1 59E28F97
 P 9500 800
-F 0 "#PWR09" H 9500 650 50  0001 C CNN
+F 0 "#PWR13" H 9500 650 50  0001 C CNN
 F 1 "+3.3V" H 9500 940 50  0000 C CNN
 F 2 "" H 9500 800 50  0001 C CNN
@@
 	9500 1100 9500 800
 $Comp
-L GND #PWR010
+L GND #PWR14
 U 1 1 59E29073
 P 9500 2100
-F 0 "#PWR010" H 9500 1850 50  0001 C CNN
+F 0 "#PWR14" H 9500 1850 50  0001 C CNN
 F 1 "GND" H 9500 1950 50  0000 C CNN
 F 2 "" H 9500 2100 50  0001 C CNN
@@
 	5150 3350 5150 3550
 $Comp
-L GND #PWR011
+L GND #PWR5
 U 1 1 59E30F3C
 P 5150 3550
-F 0 "#PWR011" H 5150 3300 50  0001 C CNN
+F 0 "#PWR5" H 5150 3300 50  0001 C CNN
 F 1 "GND" H 5150 3400 50  0000 C CNN
 F 2 "" H 5150 3550 50  0001 C CNN
@@
 	6100 3350 6100 3550
 $Comp
-L GND #PWR012
+L GND #PWR8
 U 1 1 59F090C3
 P 6100 3550
-F 0 "#PWR012" H 6100 3300 50  0001 C CNN
+F 0 "#PWR8" H 6100 3300 50  0001 C CNN
 F 1 "GND" H 6100 3400 50  0000 C CNN
 F 2 "" H 6100 3550 50  0001 C CNN
@@
 $EndComp
 $Comp
-L GND #PWR013
+L GND #PWR10
 U 1 1 59F9DB04
 P 7200 5850
-F 0 "#PWR013" H 7200 5600 50  0001 C CNN
+F 0 "#PWR10" H 7200 5600 50  0001 C CNN
 F 1 "GND" H 7200 5700 50  0000 C CNN
 F 2 "" H 7200 5850 50  0001 C CNN
@@
 $EndComp
 $Comp
-L +3.3V #PWR014
+L +3.3V #PWR7
 U 1 1 5A117D1F
 P 5200 5700
-F 0 "#PWR014" H 5200 5550 50  0001 C CNN
+F 0 "#PWR7" H 5200 5550 50  0001 C CNN
 F 1 "+3.3V" H 5200 5840 50  0000 C CNN
 F 2 "" H 5200 5700 50  0001 C CNN
@@
 IO33
 $Comp
-L GND #PWR015
+L GND #PWR6
 U 1 1 5A1181BF
 P 5200 5100
-F 0 "#PWR015" H 5200 4850 50  0001 C CNN
+F 0 "#PWR6" H 5200 4850 50  0001 C CNN
 F 1 "GND" H 5200 4950 50  0000 C CNN
 F 2 "" H 5200 5100 50  0001 C CNN
@@
 Text Label 5350 6100 2    60   ~ 0
 IO18
+Wire Wire Line
+	6750 4150 7150 4150
+Wire Wire Line
+	6750 4250 7400 4250
+Text Label 6750 4150 0    60   ~ 0
+IO19
+Text Label 6750 4250 0    60   ~ 0
+IO18
+$Comp
+L R R1
+U 1 1 5A2FC542
+P 7150 3900
+F 0 "R1" V 7230 3900 50  0000 C CNN
+F 1 "4K7" V 7050 3900 50  0000 C CNN
+F 2 "Resistors_SMD:R_0603_HandSoldering" V 7080 3900 50  0001 C CNN
+F 3 "" H 7150 3900 50  0001 C CNN
+	1    7150 3900
+	1    0    0    -1
+$EndComp
+$Comp
+L R R2
+U 1 1 5A2FCEED
+P 7400 3900
+F 0 "R2" V 7480 3900 50  0000 C CNN
+F 1 "4K7" V 7300 3900 50  0000 C CNN
+F 2 "Resistors_SMD:R_0603_HandSoldering" V 7330 3900 50  0001 C CNN
+F 3 "" H 7400 3900 50  0001 C CNN
+	1    7400 3900
+	1    0    0    -1
+$EndComp
+$Comp
+L +3.3V #PWR11
+U 1 1 5A2FD210
+P 7600 3650
+F 0 "#PWR11" H 7600 3500 50  0001 C CNN
+F 1 "+3.3V" H 7600 3790 50  0000 C CNN
+F 2 "" H 7600 3650 50  0001 C CNN
+F 3 "" H 7600 3650 50  0001 C CNN
+	1    7600 3650
+	1    0    0    -1
+$EndComp
+Wire Wire Line
+	7150 4150 7150 4050
+Wire Wire Line
+	7400 4250 7400 4050
+Wire Wire Line
+	7150 3750 7150 3700
+Wire Wire Line
+	7150 3700 7600 3700
+Wire Wire Line
+	7600 3700 7600 3650
+Wire Wire Line
+	7400 3750 7400 3700
+Connection ~ 7400 3700
 $EndSCHEMATC
